File: kicad/KP580/KP580/KP580.kicad_pcb (KiCad board)
At the start: 2 copper layers, 52 parts, among them J1 POWER, SW1 RESET, Y1 500KHz

Commit message: Генератор курсовых работ
Parts:
- added JP5: Frequency, Connector_PinHeader_2.54mm:PinHeader_2x01_P2.54mm_Vertical, F.Cu at (246.4, 80.0)
- added JP6: ~Frequency, Jumper:SolderJumper-2_P1.3mm_Open_RoundedPad1.0x1.5mm, F.Cu at (228.6, 8.89)
Connections:
- DD1 pad 4: F0 -> Net-(DD1-Pad4)
- DD1 pad 5: F0 -> Net-(DD1-Pad4)
- DD1 pad 6: ~F0 -> Net-(DD1-Pad6)
- R19 pad 1: F0 -> Net-(DD1-Pad4)
- Y1 pad 2: F0 -> Net-(DD1-Pad4)
