File: kicad/KP580/KP580/KP580.sch (KiCad schematic (older format))
At the start: 52 parts, among them J1 POWER, SW1 RESET, Y1 500KHz

Commit message: Генератор курсовых работ
Parts:
- added JP5: Frequency, Connector_PinHeader_2.54mm:PinHeader_2x01_P2.54mm_Vertical, symbol Device:Jumper
- added JP6: ~Frequency, Jumper:SolderJumper-2_P1.3mm_Open_RoundedPad1.0x1.5mm, symbol Jumper:SolderJumper_2_Open
- added TP1: +12V, TestPoint:TestPoint_Pad_D1.5mm, symbol Connector:TestPoint
- added TP2: +5V, TestPoint:TestPoint_Pad_D1.5mm, symbol Connector:TestPoint
Connections:
- wire segments 169 -> 173
Other:
- note added: "Pastor"
- moved on the sheet: DD1G, DD2C, DD3C, DD4C, DD5G, R19
