File: kicad/beacon/beacon.kicad_pcb (KiCad board)
At the start: 2 copper layers, 89.9 x 48.8 mm, 55 parts, among them J1 USB_B_Mini, K1 G5V-2, P2 Power +5V, P3 PIC Programm, P4 GPS, P5 COM, Q1 2N3904, Q2 2N3904, Q3 BS170, Q4 BS170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

Commit message: ABB логирование JSON
Parts:
- C1, C3: value 100nF -> 22pF
- R10, R9: value 4K7 -> 2K2
- R7: value 1K -> 470
