File: kicad/beacon/beacon.sch (KiCad schematic (older format))
At the start: 55 parts, among them J1 USB_B_Mini, K1 G5V-2, P2 Power +5V, P3 PIC Programm, P4 GPS, P5 COM, Q1 2N3904, Q2 2N3904, Q3 BS170, Q4 BS170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

Commit message: ABB логирование JSON
Parts:
- C1, C3: value 100nF -> 22pF
- R10, R9: value 4K7 -> 2K2
- R7: value 1K -> 470
Changed lines of the file:
@@
 P 4810 1180
 F 0 "R7" V 4603 1180 50  0000 C CNN
-F 1 "1K" V 4694 1180 50  0000 C CNN
+F 1 "470" V 4694 1180 50  0000 C CNN
 F 2 "Resistor_SMD:R_1206_3216Metric" V 4740 1180 50  0001 C CNN
 F 3 "~" H 4810 1180 50  0001 C CNN
@@
 P 1420 3750
 F 0 "C1" H 1535 3796 50  0000 L CNN
-F 1 "100nF" H 1535 3705 50  0000 L CNN
+F 1 "22pF" H 1535 3705 50  0000 L CNN
 F 2 "Capacitor_SMD:C_1206_3216Metric" H 1458 3600 50  0001 C CNN
 F 3 "~" H 1420 3750 50  0001 C CNN
@@
 P 1770 3750
 F 0 "C3" H 1885 3796 50  0000 L CNN
-F 1 "100nF" H 1885 3705 50  0000 L CNN
+F 1 "22pF" H 1885 3705 50  0000 L CNN
 F 2 "Capacitor_SMD:C_1206_3216Metric" H 1808 3600 50  0001 C CNN
 F 3 "~" H 1770 3750 50  0001 C CNN
@@
 P 6270 2960
 F 0 "R9" H 6340 3006 50  0000 L CNN
-F 1 "4K7" H 6340 2915 50  0000 L CNN
+F 1 "2K2" H 6340 2915 50  0000 L CNN
 F 2 "Resistor_SMD:R_1206_3216Metric" V 6200 2960 50  0001 C CNN
 F 3 "~" H 6270 2960 50  0001 C CNN
@@
 P 6260 3590
 F 0 "R10" H 6330 3636 50  0000 L CNN
-F 1 "4K7" H 6330 3545 50  0000 L CNN
+F 1 "2K2" H 6330 3545 50  0000 L CNN
 F 2 "Resistor_SMD:R_1206_3216Metric" V 6190 3590 50  0001 C CNN
 F 3 "~" H 6260 3590 50  0001 C CNN
